File: pcb/main/main.kicad_pcb (KiCad board)
At the start: 2 copper layers, 17 parts, among them P1 LD+, P2 LD-, P3 AC-A, P4 AC-B, P5 SPK+, P6 SPK-, Q1 PN2222A, U1 7805, U2 arduino_mini, U3 somo-ii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

Commit message: Misc
Parts:
- C1: value CP -> 2200uF
- D1, D2: value D -> 1N4007
- R1: value R -> 1k
- R2: value R -> 1.6k
- U4: value OPTO-TRANSISTOR -> 4N35
Other:
- board text added: "Chatons Corp 2017 - Sonnette MP3"
Changed lines of the file:
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@@
     (links 27)
     (no_connects 0)
-    (area 49.499999 49.499999 160.500001 120.500001)
+    (area 49.499999 49.499999 160.500001 100.500001)
     (thickness 1.6)
-    (drawings 4)
+    (drawings 5)
     (tracks 110)
     (zones 0)
@@
     (visible_elements FFFFFF7F)
     (pcbplotparams
-      (layerselection 0x00030_80000001)
+      (layerselection 0x00000_80000000)
       (usegerberextensions false)
       (excludeedgelayer true)
@@
       (psnegative false)
       (psa4output false)
-      (plotreference true)
-      (plotvalue true)
+      (plotreference false)
+      (plotvalue false)
       (plotinvisibletext false)
       (padsonsilk false)
       (subtractmaskfromsilk false)
-      (outputformat 1)
-      (mirror false)
+      (outputformat 4)
+      (mirror true)
       (drillshape 1)
       (scaleselection 1)
@@
       (effects (font (size 1 1) (thickness 0.15)))
     )
-    (fp_text value D (at 4.37134 -3.55854 180) (layer F.Fab)
+    (fp_text value 1N4007 (at 5 0 180) (layer F.Fab)
       (effects (font (size 1 1) (thickness 0.15)))
     )
@@
       (effects (font (size 1 1) (thickness 0.15)))
     )
-    (fp_text value D (at 4.37134 -3.55854 180) (layer F.Fab)
+    (fp_text value 1N4007 (at 5.3 -0.2 180) (layer F.Fab)
       (effects (font (size 1 1) (thickness 0.15)))
     )
@@
     (descr "TO-18, 3Pin,")
     (tags "TO-18, 3Pin,")
-    (fp_text reference Q1 (at 0.254 -4.826 270) (layer F.SilkS)
-      (effects (font (size 1 1) (thickness 0.15)))
-    )
-    (fp_text value PN2222A (at 0 4.826 270) (layer F.Fab)
+    (fp_text reference Q1 (at 3.8 1.2 360) (layer F.SilkS)
+      (effects (font (size 1 1) (thickness 0.15)))
+    )
+    (fp_text value PN2222A (at 5.7 -0.3 360) (layer F.Fab)
       (effects (font (size 1 1) (thickness 0.15)))
     )
@@
     (descr "Resistor, Axial,  RM 10mm, 1/3W")
     (tags "Resistor Axial RM 10mm 1/3W")
-    (fp_text reference R1 (at 5.32892 -3.50012 90) (layer F.SilkS)
-      (effects (font (size 1 1) (thickness 0.15)))
-    )
-    (fp_text value R (at 5.08 3.81 90) (layer F.Fab)
+    (fp_text reference R1 (at 5.2 -0.5 90) (layer F.SilkS)
+      (effects (font (size 1 1) (thickness 0.15)))
+    )
+    (fp_text value 1k (at 5.1 1 90) (layer F.Fab)
       (effects (font (size 1 1) (thickness 0.15)))
     )
@@
     (descr "Resistor, Axial,  RM 10mm, 1/3W")
     (tags "Resistor Axial RM 10mm 1/3W")
-    (fp_text reference R2 (at 5.32892 -3.50012 270) (layer F.SilkS)
-      (effects (font (size 1 1) (thickness 0.15)))
-    )
-    (fp_text value R (at 5.08 3.81 270) (layer F.Fab)
+    (fp_text reference R2 (at 4.9 0 270) (layer F.SilkS)
+      (effects (font (size 1 1) (thickness 0.15)))
+    )
+    (fp_text value 1.6k (at 4.8 1.5 270) (layer F.Fab)
       (effects (font (size 1 1) (thickness 0.15)))
     )
@@
     (descr "32-lead dip package, row spacing 15.24 mm (600 mils), longer pads")
     (tags "dil dip 2.54 600")
-    (fp_text reference U2 (at 0 -5.22 90) (layer F.SilkS)
-      (effects (font (size 1 1) (thickness 0.15)))
-    )
-    (fp_text value arduino_mini (at 0 -3.72 90) (layer F.Fab)
+    (fp_text reference U2 (at 6.2 29.5 180) (layer F.SilkS)
+      (effects (font (size 1 1) (thickness 0.15)))
+    )
+    (fp_text value arduino_mini (at 4.7 28.8 180) (layer F.Fab)
       (effects (font (size 1 1) (thickness 0.15)))
     )
@@
       (effects (font (size 1 1) (thickness 0.15)))
     )
-    (fp_text value OPTO-TRANSISTOR (at 0 -3.72) (layer F.Fab)
+    (fp_text value 4N35 (at 3.9 6.5) (layer F.Fab)
       (effects (font (size 1 1) (thickness 0.15)))
     )
@@
       (effects (font (size 1 1) (thickness 0.15)))
     )
-    (fp_text value CP (at 24 9.3) (layer F.Fab)
+    (fp_text value 2200uF (at 24 9.3) (layer F.Fab)
       (effects (font (size 1 1) (thickness 0.15)))
     )
@@
     (descr "24-lead dip package, row spacing 15.24 mm (600 mils), longer pads")
     (tags "dil dip 2.54 600")
-    (fp_text reference U3 (at 0 -5.22 180) (layer F.SilkS)
-      (effects (font (size 1 1) (thickness 0.15)))
-    )
-    (fp_text value somo-ii (at 0 -3.72 180) (layer F.Fab)
+    (fp_text reference U3 (at 7.5 9.9 180) (layer F.SilkS)
+      (effects (font (size 1 1) (thickness 0.15)))
+    )
+    (fp_text value somo-ii (at 7.1 8.1 180) (layer F.Fab)
       (effects (font (size 1 1) (thickness 0.15)))
     )
@@
     (descr "TO-220, Neutral, Horizontal, Large Pads,")
     (tags "TO-220, Neutral, Horizontal, Large Pads,")
-    (fp_text reference U1 (at 0.24892 -22.84984 270) (layer F.SilkS)
-      (effects (font (size 1 1) (thickness 0.15)))
-    )
-    (fp_text value 7805 (at -0.20066 4.24942 270) (layer F.Fab)
+    (fp_text reference U1 (at -0.1 -9.1 270) (layer F.SilkS)
+      (effects (font (size 1 1) (thickness 0.15)))
+    )
+    (fp_text value 7805 (at 0 -6.9 270) (layer F.Fab)
       (effects (font (size 1 1) (thickness 0.15)))
     )
@@
     (descr "Film Capacitor Length 13 x Width 4mm, Pitch 10mm")
     (tags Capacitor)
-    (fp_text reference C2 (at 5 -3.25 270) (layer F.SilkS)
-      (effects (font (size 1 1) (thickness 0.15)))
-    )
-    (fp_text value C (at 5 3.25 270) (layer F.Fab)
+    (fp_text reference C2 (at 4.9 -1 270) (layer F.SilkS)
+      (effects (font (size 1 1) (thickness 0.15)))
+    )
+    (fp_text value C (at 4.8 1.5 270) (layer F.Fab)
       (effects (font (size 1 1) (thickness 0.15)))
     )
@@
   (module Wire_Pads:Big_Square_Pad_3mm_1mmDrill (layer F.Cu)
     (at 62.7 80.8 90)
-    (fp_text reference P1 (at 0 2.54 90) (layer F.SilkS)
-      (effects (font (size 1 1) (thickness 0.15)))
-    )
-    (fp_text value LD+ (at 0 -2.54 90) (layer F.Fab)
+    (fp_text reference P1 (at -1.8 -4.5 180) (layer F.SilkS)
+      (effects (font (size 1 1) (thickness 0.15)))
+    )
+    (fp_text value LD+ (at -0.2 -4 180) (layer F.Fab)
       (effects (font (size 1 1) (thickness 0.15)))
     )
@@
   (module Wire_Pads:Big_Square_Pad_3mm_1mmDrill (layer F.Cu)
     (at 62.7 86.4 180)
-    (fp_text reference P2 (at 0 2.54 180) (layer F.SilkS)
-      (effects (font (size 1 1) (thickness 0.15)))
-    )
-    (fp_text value LD- (at 0 -2.54 180) (layer F.Fab)
+    (fp_text reference P2 (at 4.2 -0.8 180) (layer F.SilkS)
+      (effects (font (size 1 1) (thickness 0.15)))
+    )
+    (fp_text value LD- (at 3.7 0.9 180) (layer F.Fab)
       (effects (font (size 1 1) (thickness 0.15)))
     )
@@
     (pad 1 thru_hole rect (at 0 0) (size 3 3) (drill 1) (layers *.Cu *.Mask F.SilkS)
       (net 47 "Net-(P6-Pad1)"))
+  )
+  (gr_text "      Chatons Corp\n2017 - Sonnette MP3" (at 99.3 65.9) (layer B.Cu)
+    (effects (font (size 1.5 1.5) (thickness 0.375)) (justify mirror))
   )
   (gr_line (start 50 50) (end 50 100) (angle 90) (layer F.Fab) (width 1))
@@
   (segment (start 111.3 81.8) (end 126.5 81.8) (width 1) (layer B.Cu) (net 26))
   (segment (start 110.26 80.76) (end 111.3 81.8) (width 1) (layer B.Cu) (net 26))
-  (segment (start 78.92 85.64) (end 81.16 85.64) (width 1) (layer B.Cu) (net 27) (status 400000))
-  (segment (start 107.72 80.38) (end 107.72 76.66) (width 1) (layer B.Cu) (net 27) (status 800000))
+  (segment (start 78.92 85.64) (end 81.16 85.64) (width 1) (layer B.Cu) (net 27))
+  (segment (start 107.72 80.38) (end 107.72 76.66) (width 1) (layer B.Cu) (net 27))
   (segment (start 104.2 83.9) (end 107.72 80.38) (width 1) (layer B.Cu) (net 27))
   (segment (start 82.9 83.9) (end 104.2 83.9) (width 1) (layer B.Cu) (net 27))
@@
     (connect_pads (clearance 1))
     (min_thickness 0.508)
-    (fill yes (arc_segments 16) (thermal_gap 0.508) (thermal_bridge_width 2) (smoothing chamfer))
+    (fill yes (mode segment) (arc_segments 32) (thermal_gap 0.508) (thermal_bridge_width 2) (smoothing chamfer) (radius 0.508))
     (polygon
       (pts
