File: pcb/main/main.sch (KiCad schematic (older format))
At the start: 17 parts, among them P1 LD+, P2 LD-, P3 AC-A, P4 AC-B, P5 SPK+, P6 SPK-, Q1 PN2222A, U1 7805, U2 arduino_mini, U3 somo-ii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

Commit message: Misc
Parts:
- C1: value CP -> 2200uF
- D1, D2: value D -> 1N4007
- R1: value R -> 1k
- R2: value R -> 1.6k
- U4: value OPTO-TRANSISTOR -> 4N35
Changed lines of the file:
@@
 P 2100 3000
 F 0 "D1" H 2100 3100 50  0000 C CNN
-F 1 "D" H 2100 2900 50  0000 C CNN
+F 1 "1N4007" H 2100 2900 50  0000 C CNN
 F 2 "Diodes_ThroughHole:Diode_DO-41_SOD81_Horizontal_RM10" H 2100 3000 50  0001 C CNN
 F 3 "" H 2100 3000 50  0000 C CNN
@@
 P 1900 5150
 F 0 "D2" H 1900 5250 50  0000 C CNN
-F 1 "D" H 1900 5050 50  0000 C CNN
+F 1 "1N4007" H 1900 5050 50  0000 C CNN
 F 2 "Diodes_ThroughHole:Diode_DO-41_SOD81_Horizontal_RM10" H 1900 5150 50  0001 C CNN
 F 3 "" H 1900 5150 50  0000 C CNN
@@
 P 4000 4300
 F 0 "U4" H 3800 4500 50  0000 L CNN
-F 1 "OPTO-TRANSISTOR" H 3800 4100 50  0000 L CNN
+F 1 "4N35" H 3800 4100 50  0000 L CNN
 F 2 "Housings_DIP:DIP-6_W7.62mm_LongPads" H 3800 4100 50  0001 L CIN
 F 3 "" H 4000 4300 50  0000 L CNN
@@
 P 2350 4400
 F 0 "C1" H 2375 4500 50  0000 L CNN
-F 1 "CP" H 2375 4300 50  0000 L CNN
+F 1 "2200uF" H 2375 4300 50  0000 L CNN
 F 2 "Capacitors_ThroughHole:C_Axial_D16_L40_P48" H 2388 4250 50  0001 C CNN
 F 3 "" H 2350 4400 50  0000 C CNN
@@
 P 2100 4550
 F 0 "R2" V 2180 4550 50  0000 C CNN
-F 1 "R" V 2100 4550 50  0000 C CNN
+F 1 "1.6k" V 2100 4550 50  0000 C CNN
 F 2 "Resistors_ThroughHole:Resistor_Horizontal_RM10mm" V 2030 4550 50  0001 C CNN
 F 3 "" H 2100 4550 50  0000 C CNN
@@
 P 9600 3850
 F 0 "R1" V 9680 3850 50  0000 C CNN
-F 1 "R" V 9600 3850 50  0000 C CNN
+F 1 "1k" V 9600 3850 50  0000 C CNN
 F 2 "Resistors_ThroughHole:Resistor_Horizontal_RM10mm" V 9530 3850 50  0001 C CNN
 F 3 "" H 9600 3850 50  0000 C CNN
